File: Analog_Sensing.kicad_sch (KiCad schematic)
At the start: 21 parts

Commit message: revision 4
Parts:
- removed TP2: TestPoint, TestPoint:TestPoint_Pad_D2.0mm, symbol Connector:TestPoint
- C19: footprint Capacitor_SMD:C_0603_1608Metric -> Capacitor_SMD:C_0402_1005Metric
- C25: footprint Capacitor_SMD:C_0603_1608Metric -> Capacitor_SMD:C_0402_1005Metric; now not fitted; now left out of the parts list
- D9: now not fitted; now left out of the parts list
- R23, R24, R26, R27, R37, R39, R41, R44, R47, R50: footprint Resistor_SMD:R_0603_1608Metric -> Resistor_SMD:R_0402_1005Metric
- R29, R53: footprint Resistor_SMD:R_0603_1608Metric -> Resistor_SMD:R_0402_1005Metric; LCSC (none) -> C409665
- R56, R57, R62: footprint Resistor_SMD:R_0603_1608Metric -> Resistor_SMD:R_0402_1005Metric; now not fitted; now left out of the parts list
- TP1: now left out of the parts list
Connections:
- net VDDA renamed VDD
