File: Inputs_out_Puts.kicad_sch (KiCad schematic)
At the start: 37 parts, among them J1 Conn_01x03_Pin, J14 USB_C_Receptacle_USB2.0, J4 Conn_01x02_Female, J8 Conn_01x03_MountingPin, J9 Conn_01x06_MountingPin, SW1 SW_MEC_5G, U1 TCAN330, U2 TPS709-5

Commit message: revision 4
Parts:
- removed C15: 100nF, Capacitor_SMD:C_0603_1608Metric, symbol Device:C
- removed J9: Conn_01x06_MountingPin, Connector_JST:JST_SH_BM06B-SRSS-TB_1x06-1MP_P1.00mm_Vertical, symbol Connector_Generic_MountingPin:Conn_01x06_MountingPin
- removed R8: 100k, Resistor_SMD:R_0603_1608Metric, symbol Device:R
- removed SW1: SW_MEC_5G, mystuff:SW_SPST_TS-1187A-B, symbol Switch:SW_Push
- removed TP10: TestPoint, TestPoint:TestPoint_Pad_D1.5mm, symbol Connector:TestPoint
- removed TP7, TP8, TP9: TestPoint, TestPoint:TestPoint_Pad_D1.0mm, symbol Connector:TestPoint
- removed U1: TCAN330, Package_SO:SOIC-8_3.9x4.9mm_P1.27mm, symbol Interface_CAN_LIN:TCAN330
- removed U2: TPS709-5, Package_TO_SOT_SMD:TSOT-23-5, symbol mystuff:TPS709-5
- added C3: 2.2uf, Capacitor_SMD:C_1206_3216Metric, symbol Device:C
- added J2: Conn_01x12_MountingPin, Connector_FFC-FPC:TE_1-1734839-2_1x12-1MP_P0.5mm_Horizontal, symbol Connector_Generic_MountingPin:Conn_01x12_MountingPin
- added J3: Conn_01x08_MountingPin, Connector_JST:JST_SH_BM08B-SRSS-TB_1x08-1MP_P1.00mm_Vertical, symbol Connector_Generic_MountingPin:Conn_01x08_MountingPin
- added J5: Conn_01x03_MountingPin, Connector_JST:JST_SH_BM03B-SRSS-TB_1x03-1MP_P1.00mm_Vertical, symbol Connector_Generic_MountingPin:Conn_01x03_MountingPin
- added J6: Conn_01x06_MountingPin, Connector_JST:JST_SH_BM06B-SRSS-TB_1x06-1MP_P1.00mm_Vertical, symbol Connector_Generic_MountingPin:Conn_01x06_MountingPin
- added U2: TJA1057T/1Z, Package_SO:SOIC-8_3.9x4.9mm_P1.27mm, symbol Interface_CAN_LIN:TJA1051T
- added U3: TC1017-xCT, Package_TO_SOT_SMD:SOT-23-5, symbol Regulator_Linear:TC1017-xCT
- C14: footprint Capacitor_SMD:C_0603_1608Metric -> Capacitor_SMD:C_0402_1005Metric; LCSC Part C15849 -> (none)
- C41: footprint Capacitor_SMD:C_0603_1608Metric -> Capacitor_SMD:C_0402_1005Metric
- J1: footprint mystuff:flat_3 -> Connector_JST:JST_XH_B3B-XH-AM_1x03_P2.50mm_Vertical
- R19: footprint Resistor_SMD:R_0603_1608Metric -> Resistor_SMD:R_0402_1005Metric; LCSC Part C23186 -> (none)
- R20, R5, R6, R98: footprint Resistor_SMD:R_0603_1608Metric -> Resistor_SMD:R_0402_1005Metric
- R7: value 220 -> 110; footprint Resistor_SMD:R_0603_1608Metric -> Resistor_SMD:R_0402_1005Metric
- R99: value 10k -> 10K; footprint Resistor_SMD:R_0603_1608Metric -> Resistor_SMD:R_0402_1005Metric
- renumbered D4 to D4_white1, D6 to D6_Yellow1
Connections:
- net +5V: now also U3.5 (VOUT)
- net CAN_SHDN: now also R99.1; no longer R99.2
- net FDCAN1_RX/BOOT_0: now also U2.4 (RXD)
- net FDCAN1_TX: now also U2.1 (TXD)
- net GND: now also C3.2, J2.10 (Pin_10), J2.11 (Pin_11), J2.8 (Pin_8), J2.MP (MountPin), J3.8 (Pin_8), J3.MP (MountPin), J5.3 (Pin_3), J5.MP (MountPin), J6.1 (Pin_1), J6.MP (MountPin), U2.2 (GND), U3.2 (GND)
- net GPIO_PA10: now also J3.1 (Pin_1)
- net I2C2_SCL: now also J3.3 (Pin_3)
- net I2C2_SDA: now also J3.2 (Pin_2)
- net SPI1_MISO: now also J3.5 (Pin_5)
- net SPI1_MOSI: now also J3.4 (Pin_4)
- net SPI1_SCK: now also J3.6 (Pin_6)
- net VCC: now also U3.1 (VIN), U3.3 (~{SHDN})
- net VDD: now also U2.3 (VCC)
- net VM: now also C3.1
- net at J8.1 (Pin_1), R98.2: now also J5.1 (Pin_1), U2.6 (CANL)
- net at J8.2 (Pin_2), R98.1: now also J5.2 (Pin_2), U2.7 (CANH)
- net at JP1.2 (C): now also J3.7 (Pin_7)
- new net: R99.2, U2.8 (S)
- new net +3V3: J6.2 (Pin_2)
- new net 24VIN: J2.12 (Pin_12)
- new net 5Vout: J2.9 (Pin_9)
- new net CS: J2.4 (Pin_4)
- new net HA: J6.3 (Pin_3)
- new net HB: J6.4 (Pin_4)
- new net HC: J6.5 (Pin_5)
- new net MISO: J2.3 (Pin_3)
- new net MOSI: J2.2 (Pin_2)
- new net PS1: J2.5 (Pin_5), J2.7 (Pin_7)
- new net PS2: J2.6 (Pin_6)
- new net SCK: J2.1 (Pin_1)
- no-connect marks 3 -> 2
Other:
- note added: "ENC_A"
- note added: "ENC_B"
- note added: "ENC_I"
- moved on the sheet: C14
