File: Power_Stage.kicad_sch (KiCad schematic)
At the start: 25 parts, among them Q1 Q_NMOS_GDS, Q2 Q_NMOS_GDS, Q3 Q_NMOS_GDS, Q4 Q_NMOS_GDS, Q5 Q_NMOS_GDS, Q6 Q_NMOS_GDS

Commit message: revision 4
Parts:
- Q1, Q2, Q3, Q4, Q5, Q6: footprint my_stuff:DFN-8-1EP_6x5mm_P1.27mm_EP4x4mm -> mystuff:DFN-8-1EP_6x5mm_P1.27mm_EP4x4mm
- R1, R13, R17, R18, R25, R4: footprint Resistor_SMD:R_0603_1608Metric -> Resistor_SMD:R_0402_1005Metric; LCSC Part C23140 -> (none)
Changed lines of the file:
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@@
       (effects (font (size 1.27 1.27)))
     )
-    (property "Footprint" "Resistor_SMD:R_0603_1608Metric" (at 76.2 56.642 90)
+    (property "Footprint" "Resistor_SMD:R_0402_1005Metric" (at 76.2 56.642 90)
       (effects (font (size 1.27 1.27)) hide)
     )
     (property "Datasheet" "~" (at 76.2 58.42 0)
-      (effects (font (size 1.27 1.27)) hide)
-    )
-    (property "LCSC Part" "C23140" (at 76.2 58.42 90)
       (effects (font (size 1.27 1.27)) hide)
     )
@@
       (effects (font (size 1.27 1.27)))
     )
-    (property "Footprint" "Resistor_SMD:R_0603_1608Metric" (at 76.2 90.932 90)
+    (property "Footprint" "Resistor_SMD:R_0402_1005Metric" (at 76.2 90.932 90)
       (effects (font (size 1.27 1.27)) hide)
     )
     (property "Datasheet" "~" (at 76.2 92.71 0)
-      (effects (font (size 1.27 1.27)) hide)
-    )
-    (property "LCSC Part" "C23140" (at 76.2 92.71 90)
       (effects (font (size 1.27 1.27)) hide)
     )
@@
       (effects (font (size 1.27 1.27)) (justify left))
     )
-    (property "Footprint" "my_stuff:DFN-8-1EP_6x5mm_P1.27mm_EP4x4mm" (at 99.06 55.88 0)
+    (property "Footprint" "mystuff:DFN-8-1EP_6x5mm_P1.27mm_EP4x4mm" (at 99.06 55.88 0)
       (effects (font (size 1.27 1.27)) hide)
     )
@@
       (effects (font (size 1.27 1.27)))
     )
-    (property "Footprint" "Resistor_SMD:R_0603_1608Metric" (at 224.79 88.392 90)
+    (property "Footprint" "Resistor_SMD:R_0402_1005Metric" (at 224.79 88.392 90)
       (effects (font (size 1.27 1.27)) hide)
     )
     (property "Datasheet" "~" (at 224.79 90.17 0)
-      (effects (font (size 1.27 1.27)) hide)
-    )
-    (property "LCSC Part" "C23140" (at 224.79 90.17 90)
       (effects (font (size 1.27 1.27)) hide)
     )
@@
       (effects (font (size 1.27 1.27)))
     )
-    (property "Footprint" "Resistor_SMD:R_0603_1608Metric" (at 146.05 88.392 90)
+    (property "Footprint" "Resistor_SMD:R_0402_1005Metric" (at 146.05 88.392 90)
       (effects (font (size 1.27 1.27)) hide)
     )
     (property "Datasheet" "~" (at 146.05 90.17 0)
-      (effects (font (size 1.27 1.27)) hide)
-    )
-    (property "LCSC Part" "C23140" (at 146.05 90.17 90)
       (effects (font (size 1.27 1.27)) hide)
     )
@@
       (effects (font (size 1.27 1.27)) (justify left))
     )
-    (property "Footprint" "my_stuff:DFN-8-1EP_6x5mm_P1.27mm_EP4x4mm" (at 168.91 53.34 0)
+    (property "Footprint" "mystuff:DFN-8-1EP_6x5mm_P1.27mm_EP4x4mm" (at 168.91 53.34 0)
       (effects (font (size 1.27 1.27)) hide)
     )
@@
       (effects (font (size 1.27 1.27)))
     )
-    (property "Footprint" "Resistor_SMD:R_0603_1608Metric" (at 224.79 54.102 90)
+    (property "Footprint" "Resistor_SMD:R_0402_1005Metric" (at 224.79 54.102 90)
       (effects (font (size 1.27 1.27)) hide)
     )
     (property "Datasheet" "~" (at 224.79 55.88 0)
-      (effects (font (size 1.27 1.27)) hide)
-    )
-    (property "LCSC Part" "C23140" (at 224.79 55.88 90)
       (effects (font (size 1.27 1.27)) hide)
     )
@@
       (effects (font (size 1.27 1.27)) (justify left))
     )
-    (property "Footprint" "my_stuff:DFN-8-1EP_6x5mm_P1.27mm_EP4x4mm" (at 168.91 87.63 0)
+    (property "Footprint" "mystuff:DFN-8-1EP_6x5mm_P1.27mm_EP4x4mm" (at 168.91 87.63 0)
       (effects (font (size 1.27 1.27)) hide)
     )
@@
       (effects (font (size 1.27 1.27)) (justify left))
     )
-    (property "Footprint" "my_stuff:DFN-8-1EP_6x5mm_P1.27mm_EP4x4mm" (at 247.65 53.34 0)
+    (property "Footprint" "mystuff:DFN-8-1EP_6x5mm_P1.27mm_EP4x4mm" (at 247.65 53.34 0)
       (effects (font (size 1.27 1.27)) hide)
     )
@@
       (effects (font (size 1.27 1.27)) (justify left))
     )
-    (property "Footprint" "my_stuff:DFN-8-1EP_6x5mm_P1.27mm_EP4x4mm" (at 99.06 90.17 0)
+    (property "Footprint" "mystuff:DFN-8-1EP_6x5mm_P1.27mm_EP4x4mm" (at 99.06 90.17 0)
       (effects (font (size 1.27 1.27)) hide)
     )
@@
       (effects (font (size 1.27 1.27)) (justify left))
     )
-    (property "Footprint" "my_stuff:DFN-8-1EP_6x5mm_P1.27mm_EP4x4mm" (at 247.65 87.63 0)
+    (property "Footprint" "mystuff:DFN-8-1EP_6x5mm_P1.27mm_EP4x4mm" (at 247.65 87.63 0)
       (effects (font (size 1.27 1.27)) hide)
     )
@@
       (effects (font (size 1.27 1.27)))
     )
-    (property "Footprint" "Resistor_SMD:R_0603_1608Metric" (at 146.05 54.102 90)
+    (property "Footprint" "Resistor_SMD:R_0402_1005Metric" (at 146.05 54.102 90)
       (effects (font (size 1.27 1.27)) hide)
     )
@@
       (effects (font (size 1.27 1.27)) hide)
     )
-    (property "LCSC Part" "C23140" (at 146.05 55.88 90)
-      (effects (font (size 1.27 1.27)) hide)
-    )
